File: esprelayboard/esprelayboard.brd (EAGLE design)
At the start: 67.2 x 51.6 mm, 95 parts, among them IC1 MP2315GJ-Z, IC4 CP2104, J1 SM06B-GHS-TB_LF__SN_, J2 SM02B-GHS-TB_LF__SN_, J4 SM06B-GHS-TB_LF__SN_, J6 SM02B-GHS-TB_LF__SN_, J7 SM02B-GHS-TB_LF__SN_, J8 SM02B-GHS-TB_LF__SN_, J9 SM02B-GHS-TB_LF__SN_, K1 G6K-2F-Y, K2 G6K-2F-Y, K4 G6K-2F-Y, Q1 MOSFET-NCHANNELAO3404A, Q2 MOSFET-NCHANNELAO3404A, Q3 MOSFET-NCHANNELAO3404A, Q5 mmbt2222, Q6 mmbt2222, U2 AP2112-3.3, U3 CCS811, X8 ESP32_WROOM32_SKINNY

Commit message: final board files
Parts:
- removed RESET: KMR2, microbuilder:BTN_KMR2_4.6X2.8
- added IO0, RST: 436331045822, 436331045822:436331045822
- moved U$38 7.57 mm to (59.2, 0.91)
Connections:
- net GND: now also IO0.2, IO0.4, RST.2, RST.4; no longer RESET.A, RESET.A'
- net GPIO0: now also IO0.1, IO0.3
- net RESET: now also RST.1, RST.3; no longer RESET.B, RESET.B'
Routing:
- net GPIO0: track 4.49 -> 63.9 mm, vias 0 -> 5
- net RESET: track 91.7 -> 92.9 mm
Other:
- outline, holes or cut-outs redrawn
- board text added: "v1.0"

Commit message: v2
Parts:
- removed D+, D-: TPB1,27, testpad:B1,27
- removed D3: (no value), diode:DO214AA
- added D6: MBR120, microbuilder:SOD-123
- C9: device rcl:140CLH-1010 -> rcl:UD-6,3X5,8_NICHICON
- D1, D2: value (none) -> MBR120; device diode:DO214AA -> microbuilder:SOD-123
- L1: device rcl:POWER-CHOKE_WE-TPC -> rcl:L2825P
- moved LED1 53.9 mm to (57.3, 29.9), turned to 0 degrees
- moved U$38 53.2 mm to (6.05, -1.02)
- moved RST 28.8 mm to (38.1, 30.9), turned to 180 degrees
- moved IO0 27.5 mm to (45.6, 30.9), turned to 180 degrees
- moved C9 27.1 mm to (46.1, 17.1), turned to 90 degrees
- moved J9 25.2 mm to (30.5, 30.1), turned to 180 degrees
- moved D5 23.0 mm to (40.4, 25.4), turned to 90 degrees
- moved U$39 21.9 mm to (65.0, 27.6)
- moved TP16 21.7 mm to (32.8, 28.8)
- moved TP17 21.5 mm to (28.4, 29.0)
- moved D1 21.4 mm to (20.3, 17.8), flipped to the bottom
- moved SJ3 21.3 mm to (43.3, 26.0)
- moved R45 19.3 mm to (37.5, 25.6), turned to 90 degrees
- moved TP18 19.0 mm to (8.53, 27.1)
- moved R10 18.9 mm to (5.64, 24.6)
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Connections:
- net D+: no longer D+.TP
- net D-: no longer D-.TP
- net N$3: now also D2.A; no longer D1.A
- net N$7: now also D1.A; no longer D2.A
- net N$8: now also D6.A; no longer D3.A
- net VBUS: now also D6.C; no longer D3.C
Routing:
- net 3.3V: track 269.8 -> 182.0 mm
- net TXD0: track 52.7 -> 129.2 mm, vias 2 -> 4
- net NEOPIX: track 84.6 -> 8.93 mm, vias 3 -> 1
- net GPIO0: track 63.9 -> 16.7 mm, vias 5 -> 1
- net RXD0: track 53.6 -> 99.3 mm, vias 2 -> 5
- net R1OA: track 69.1 -> 24.2 mm
- net N$48: track 43.9 -> 87.3 mm
- net VBUS: track 155.1 -> 117.2 mm, vias 5 -> 7
- net R1OB: track 60.0 -> 22.6 mm
- net ISO_DIN_NEG: track 49.5 -> 14.1 mm, vias 2 -> 0
- net N$9: track 49.6 -> 15.2 mm, vias 4 -> 0
- net DTR: track 66.8 -> 97.4 mm, vias 0 -> 2
- net DIN_2: track 53.7 -> 26.0 mm, vias 1 -> 3
- net VIN: track 86.9 -> 110.9 mm, vias 7 -> 2
- net DIN_1: track 52.4 -> 30.7 mm
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Other:
- board size 67.2 x 51.6 mm -> 67.5 x 33.1 mm
- board text added: "+"
- board text added: "-"
- board text added: "GPIO0"
- board text added: "ISO_IN"
- board text added: "RST"
- board text added: "v2.0"
- board text removed: "RA1"
- board text removed: "v1.0"

Commit message: bug fix
Parts:
- R24: value 100k -> 10k
- moved U$39 43.1 mm to (30.3, 2.24)
- moved D13 0.64 mm to (44.8, 3.25)
Connections:
- removed net !RST_3V: R24.2, U3.2
- removed net !WAKE_3V: R24.3, U3.7
- new net INT_CCS811: U3.3, X8.23
- new net RST_CCS811: R24.2, U3.2, X8.13
- new net WAKE_CCS811: R24.3, U3.7, X8.16
- net NEOPIX: now also X8.37; no longer X8.33
- net SDA: now also X8.33; no longer X8.37
Routing:
- net INT_CCS811: track 0.00 -> 66.4 mm, vias 0 -> 3
- net WAKE_CCS811: track 0.00 -> 60.0 mm, vias 0 -> 5
- net RST_CCS811: track 0.00 -> 47.4 mm, vias 0 -> 1
- net !WAKE_3V: track 22.5 -> 0.00 mm, vias 2 -> 0
- net !RST_3V: track 8.02 -> 0.00 mm
- net 3.3V: track 182.0 -> 185.3 mm
- net RELAY1: track 32.4 -> 35.2 mm
- net R3OD: track 37.0 -> 35.3 mm
- net N$13: track 8.06 -> 9.43 mm
- net VIN: track 110.9 -> 109.9 mm
- net NEOPIX: track 8.93 -> 7.95 mm
- net N$1: track 2.33 -> 1.80 mm
- net SDA: track 101.5 -> 102.0 mm, vias 3 -> 5
- net N$14: track 21.2 -> 21.7 mm
Other:
- outline, holes or cut-outs redrawn

Commit message: v2
Parts:
- removed C8: DSK-3R3H224U-HL, DSK-3R3H224U-HL:CAP_DSK-3R3H224U-HL
- added 3V3: SM02B-GHS-TB_LF__SN_, SM02B-GHS-TB_LF__SN_:SM02BGHSTBLFSN
- added C11: 1uF, microbuilder:0603-NO@1
- added C12: 10µF, microbuilder:0805-NO
- added R18: 100K, microbuilder:0603-NO
- added U1: AP2112-3.3, microbuilder:SOT23-5
- R3: value 5K -> 10K
- moved U$39 35.0 mm to (65.0, 5.54), turned to 270 degrees
- moved C2 29.9 mm to (56.1, 19.2), flipped to the top, turned to 270 degrees
- moved C28 29.0 mm to (56.7, 23.0), flipped to the top, turned to 90 degrees
- moved U2 22.1 mm to (53.2, 20.8), flipped to the top, turned to 0 degrees
- moved R44 19.3 mm to (53.2, 17.6), flipped to the top, turned to 180 degrees
- moved C30 16.9 mm to (52.1, 29.9), flipped to the top
- moved D13 9.66 mm to (36.3, 7.77), flipped to the top, turned to 90 degrees
- moved R43 2.85 mm to (44.4, 5.59)
- moved R24 0.53 mm to (13.8, 9.55)
- moved TP18 0.36 mm to (8.59, 27.4)
- moved U$38 0.15 mm to (5.89, -1.04)
- moved J9 0.10 mm to (30.5, 30.2)
- moved J7 0.09 mm to (39.0, 3.09)
Connections:
- new net 3.3V-2: 3V3.2, C11.1, C12.1, C30.1, IC4.5, IC4.6, IC4.7, LED1.2, R24.6, R24.7, R24.8, R46.3, U1.5, U3.6
- new net EN_U1: R18.1, U1.3
- net 3.3V: now also R3.1; no longer C30.1, C8.1, IC4.5, IC4.6, IC4.7, LED1.2, OK1.4, R24.6, R24.7, R24.8, R46.3, U3.6
- net GND: now also 3V3.1, 3V3.3, 3V3.4, C11.2, C12.2, OK1.3, U1.2; no longer C8.2, R3.1
- net ISO_DIN: now also OK1.4; no longer OK1.3
- net VBUS: now also R18.2, U1.1
Routing:
- net 3.3V-2: track 0.00 -> 145.9 mm, vias 0 -> 6
- net 3.3V: track 185.3 -> 52.4 mm, vias 9 -> 2
- net VBUS: track 117.2 -> 147.7 mm, vias 7 -> 9
- net TXD0: track 129.4 -> 105.7 mm
- net INT_CCS811: track 66.4 -> 52.7 mm
- net N$1: track 1.80 -> 9.65 mm, vias 0 -> 1
- net ISO_DIN: track 23.6 -> 28.4 mm, vias 2 -> 1
- net RESET: track 89.6 -> 94.0 mm, vias 3 -> 4
- net RXD0: track 99.2 -> 95.5 mm
- net WAKE_CCS811: track 60.0 -> 62.3 mm
- net N$9: track 15.2 -> 17.4 mm
- net PW_LED: track 3.41 -> 5.39 mm
- net RST_CCS811: track 47.4 -> 49.2 mm
- net SDA: track 102.0 -> 103.6 mm
- net EN_U1: track 0.00 -> 1.60 mm
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Other:
- board size 67.5 x 33.1 mm -> 67.3 x 33.1 mm
- board text added: "3v3"
