File: esprelayboard/esprelayboard.sch (EAGLE design)
At the start: 93 parts, among them IC1 MP2315GJ-Z, IC4 CP2104, J1 SM06B-GHS-TB_LF__SN_, J2 SM02B-GHS-TB_LF__SN_, J4 SM06B-GHS-TB_LF__SN_, J6 SM02B-GHS-TB_LF__SN_, J7 SM02B-GHS-TB_LF__SN_, J8 SM02B-GHS-TB_LF__SN_, J9 SM02B-GHS-TB_LF__SN_, K1 G6K-2F-Y, K2 G6K-2F-Y, K4 G6K-2F-Y, Q1 MOSFET-NCHANNELAO3404A, Q2 MOSFET-NCHANNELAO3404A, Q3 MOSFET-NCHANNELAO3404A, Q5 mmbt2222, Q6 mmbt2222, U2 AP2112-3.3, U3 CCS811, X8 ESP32_WROOM32_SKINNY

Commit message: final board files
Parts:
- removed RESET: KMR2, microbuilder:SWITCH_TACT_SMT4.6X2.8
- added IO0, RST: 436331045822, 436331045822:436331045822
Connections:
- net GND: now also IO0.2, IO0.4, RST.2, RST.4; no longer RESET.P, RESET.P1
- net GPIO0: now also IO0.1, IO0.3
- net RESET: now also RST.1, RST.3; no longer RESET.S, RESET.S1
Other:
- moved on the sheet: C32
Changed lines of the file:
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@@
 <setting verticaltext="up"/>
 </settings>
-<grid distance="0.01" unitdist="inch" unit="inch" style="lines" multiple="1" display="no" altdistance="0.01" altunitdist="inch" altunit="inch"/>
+<grid distance="0.1" unitdist="inch" unit="inch" style="lines" multiple="1" display="no" altdistance="0.01" altunitdist="inch" altunit="inch"/>
 <layers>
 <layer number="1" name="Top" color="4" fill="1" visible="no" active="no"/>
@@
 <parts>
 <part name="U$14" library="microbuilder" deviceset="3.3V" device=""/>
-<part name="RESET" library="microbuilder" deviceset="SWITCH_TACT_SMT" device="4.6X2.8" value="KMR2"/>
 <part name="GND20" library="supply1" deviceset="GND" device=""/>
 <part name="D13" library="microbuilder" deviceset="LED" device="0805_NOOUTLINE" value="RED"/>
@@
 <part name="C9" library="rcl" library_urn="urn:adsk.eagle:library:334" deviceset="CPOL-US" device="140CLH-1010" package3d_urn="urn:adsk.eagle:package:23391/2"/>
 <part name="U$40" library="microbuilder" deviceset="GND" device=""/>
+<part name="RST" library="436331045822" deviceset="436331045822" device=""/>
+<part name="GND1" library="supply1" deviceset="GND" device=""/>
+<part name="IO0" library="436331045822" deviceset="436331045822" device=""/>
 </parts>
 <sheets>
@@
 <attribute name="VALUE" x="84.836" y="120.396" size="1.27" layer="96"/>
 </instance>
-<instance part="RESET" gate="G$1" x="83.82" y="91.44" smashed="yes" rot="R90">
-<attribute name="NAME" x="77.47" y="88.9" size="1.27" layer="95" rot="R90"/>
-<attribute name="VALUE" x="88.9" y="88.9" size="1.27" layer="96" rot="R90"/>
-</instance>
-<instance part="GND20" gate="1" x="86.36" y="83.82" smashed="yes">
-<attribute name="VALUE" x="83.82" y="81.28" size="1.778" layer="96"/>
+<instance part="GND20" gate="1" x="81.28" y="81.28" smashed="yes">
+<attribute name="VALUE" x="78.74" y="78.74" size="1.778" layer="96"/>
 </instance>
 <instance part="D13" gate="G$1" x="96.52" y="-22.86" smashed="yes" rot="R90">
@@
 <attribute name="VALUE" x="71.12" y="10.16" size="1.016" layer="96" font="vector" ratio="15" align="center"/>
 </instance>
-<instance part="C32" gate="G$1" x="96.52" y="91.44" smashed="yes">
-<attribute name="NAME" x="94.23" y="92.69" size="1.27" layer="95" font="vector" rot="R90" align="center"/>
-<attribute name="VALUE" x="98.82" y="92.69" size="1.27" layer="96" font="vector" rot="R90" align="center"/>
-</instance>
-<instance part="U$52" gate="G$1" x="96.52" y="86.36" smashed="yes">
-<attribute name="VALUE" x="94.996" y="83.82" size="1.27" layer="96"/>
+<instance part="C32" gate="G$1" x="91.44" y="91.44" smashed="yes">
+<attribute name="NAME" x="89.15" y="92.69" size="1.27" layer="95" font="vector" rot="R90" align="center"/>
+<attribute name="VALUE" x="93.74" y="92.69" size="1.27" layer="96" font="vector" rot="R90" align="center"/>
+</instance>
+<instance part="U$52" gate="G$1" x="91.44" y="86.36" smashed="yes">
+<attribute name="VALUE" x="89.916" y="83.82" size="1.27" layer="96"/>
 </instance>
 <instance part="IC4" gate="G$1" x="149.86" y="83.82" smashed="yes">
@@
 <instance part="U$40" gate="G$1" x="-36.068" y="2.794" smashed="yes">
 <attribute name="VALUE" x="-37.592" y="0.254" size="1.27" layer="96"/>
+</instance>
+<instance part="RST" gate="G$1" x="81.28" y="91.44" smashed="yes">
+<attribute name="NAME" x="85.09" y="92.71" size="1.778" layer="95"/>
+</instance>
+<instance part="GND1" gate="1" x="99.06" y="81.28" smashed="yes">
+<attribute name="VALUE" x="96.52" y="78.74" size="1.778" layer="96"/>
+</instance>
+<instance part="IO0" gate="G$1" x="99.06" y="91.44" smashed="yes">
+<attribute name="NAME" x="102.87" y="92.71" size="1.778" layer="95"/>
+<attribute name="VALUE" x="102.87" y="88.9" size="1.778" layer="96"/>
 </instance>
 </instances>
@@
 <nets>
 <net name="GND" class="0">
-<segment>
-<pinref part="RESET" gate="G$1" pin="P"/>
-<pinref part="RESET" gate="G$1" pin="P1"/>
-<wire x1="83.82" y1="86.36" x2="86.36" y2="86.36" width="0.1524" layer="91"/>
-<pinref part="GND20" gate="1" pin="GND"/>
-<junction x="86.36" y="86.36"/>
-</segment>
 <segment>
 <pinref part="U$45" gate="G$1" pin="GND"/>
@@
 <pinref part="C9" gate="G$1" pin="-"/>
 <pinref part="U$40" gate="G$1" pin="GND"/>
+</segment>
+<segment>
+<pinref part="RST" gate="G$1" pin="2"/>
+<wire x1="76.2" y1="86.36" x2="76.2" y2="83.82" width="0.1524" layer="91"/>
+<pinref part="GND20" gate="1" pin="GND"/>
+<wire x1="76.2" y1="83.82" x2="81.28" y2="83.82" width="0.1524" layer="91"/>
+<pinref part="RST" gate="G$1" pin="4"/>
+<wire x1="81.28" y1="83.82" x2="86.36" y2="83.82" width="0.1524" layer="91"/>
+<wire x1="86.36" y1="83.82" x2="86.36" y2="86.36" width="0.1524" layer="91"/>
+<junction x="81.28" y="83.82"/>
+</segment>
+<segment>
+<pinref part="GND1" gate="1" pin="GND"/>
+<pinref part="IO0" gate="G$1" pin="2"/>
+<wire x1="93.98" y1="86.36" x2="93.98" y2="83.82" width="0.1524" layer="91"/>
+<wire x1="93.98" y1="83.82" x2="99.06" y2="83.82" width="0.1524" layer="91"/>
+<pinref part="IO0" gate="G$1" pin="4"/>
+<wire x1="104.14" y1="86.36" x2="104.14" y2="83.82" width="0.1524" layer="91"/>
+<wire x1="104.14" y1="83.82" x2="99.06" y2="83.82" width="0.1524" layer="91"/>
+<junction x="99.06" y="83.82"/>
 </segment>
 </net>
@@
 <net name="RESET" class="0">
 <segment>
-<wire x1="86.36" y1="104.14" x2="86.36" y2="96.52" width="0.1524" layer="91"/>
+<wire x1="86.36" y1="104.14" x2="86.36" y2="99.06" width="0.1524" layer="91"/>
 <label x="88.9" y="96.52" size="1.778" layer="95" rot="R90"/>
-<pinref part="RESET" gate="G$1" pin="S1"/>
-<pinref part="RESET" gate="G$1" pin="S"/>
-<wire x1="86.36" y1="96.52" x2="83.82" y2="96.52" width="0.1524" layer="91"/>
-<junction x="86.36" y="96.52"/>
 <pinref part="R46" gate="G$3" pin="2"/>
+<pinref part="RST" gate="G$1" pin="3"/>
+<pinref part="RST" gate="G$1" pin="1"/>
+<wire x1="86.36" y1="99.06" x2="86.36" y2="96.52" width="0.1524" layer="91"/>
+<wire x1="76.2" y1="96.52" x2="76.2" y2="99.06" width="0.1524" layer="91"/>
+<wire x1="76.2" y1="99.06" x2="86.36" y2="99.06" width="0.1524" layer="91"/>
+<junction x="86.36" y="99.06"/>
 </segment>
 <segment>
@@
 <segment>
 <pinref part="C32" gate="G$1" pin="1"/>
-<wire x1="96.52" y1="96.52" x2="96.52" y2="109.22" width="0.1524" layer="91"/>
-<label x="96.52" y="101.6" size="1.778" layer="95" rot="R90"/>
-<junction x="96.52" y="96.52"/>
+<wire x1="91.44" y1="96.52" x2="91.44" y2="109.22" width="0.1524" layer="91"/>
+<label x="91.44" y="101.6" size="1.778" layer="95" rot="R90"/>
+<junction x="91.44" y="96.52"/>
 </segment>
 </net>
@@
 <pinref part="X8" gate="G$1" pin="IO0/A2_1"/>
 </segment>
+<segment>
+<pinref part="IO0" gate="G$1" pin="1"/>
+<wire x1="93.98" y1="96.52" x2="93.98" y2="99.06" width="0.1524" layer="91"/>
+<pinref part="IO0" gate="G$1" pin="3"/>
+<wire x1="104.14" y1="96.52" x2="104.14" y2="99.06" width="0.1524" layer="91"/>
+<wire x1="104.14" y1="99.06" x2="93.98" y2="99.06" width="0.1524" layer="91"/>
+<label x="96.52" y="99.06" size="1.778" layer="95"/>
+</segment>
 </net>

Commit message: v2
Parts:
- removed D+, D-: TPB1,27, testpad:TPB1,27
- removed D3: (no value), diode:DIODE-DO214AA
- added D6: MBR120, microbuilder:DIODE-SCHOTTKYSOD-123
- C9: device rcl:CPOL-US140CLH-1010 -> rcl:CPOL-USUD-6,3X5,8
- D1, D2: value (none) -> MBR120; device diode:DIODE-DO214AA -> microbuilder:DIODE-SCHOTTKYSOD-123
- L1: device rcl:L-EUWE-TPC -> rcl:L-EUL2825P
Connections:
- net D+: no longer D+.TP
- net D-: no longer D-.TP
- net N$3: now also D2.A; no longer D1.A
- net N$7: now also D1.A; no longer D2.A
- net N$8: now also D6.A; no longer D3.A
- net VBUS: now also D6.C; no longer D3.C

Commit message: bug fix
Parts:
- R24: value 100k -> 10k
Connections:
- removed net !RST_3V: R24G$2.1, U3.!RST
- removed net !WAKE_3V: R24G$3.1, U3.!WAKE
- new net INT_CCS811: U3.!INT, X8.IO15/A2_3
- new net RST_CCS811: R24G$2.1, U3.!RST, X8.IO14/A2_6
- new net WAKE_CCS811: R24G$3.1, U3.!WAKE, X8.IO13/A2_4
- net NEOPIX: now also X8.IO23; no longer X8.IO21
- net SDA: now also X8.IO21; no longer X8.IO23
Changed lines of the file:
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@@
 <grid distance="0.01" unitdist="inch" unit="inch" style="lines" multiple="1" display="no" altdistance="0.01" altunitdist="inch" altunit="inch"/>
 <layers>
-<layer number="1" name="Top" color="4" fill="1" visible="yes" active="no"/>
-<layer number="16" name="Bottom" color="1" fill="1" visible="yes" active="no"/>
-<layer number="17" name="Pads" color="2" fill="1" visible="yes" active="no"/>
-<layer number="18" name="Vias" color="2" fill="1" visible="yes" active="no"/>
-<layer number="19" name="Unrouted" color="6" fill="1" visible="yes" active="no"/>
-<layer number="20" name="Dimension" color="24" fill="1" visible="yes" active="no"/>
-<layer number="21" name="tPlace" color="7" fill="1" visible="yes" active="no"/>
-<layer number="22" name="bPlace" color="7" fill="1" visible="yes" active="no"/>
-<layer number="23" name="tOrigins" color="15" fill="1" visible="yes" active="no"/>
-<layer number="24" name="bOrigins" color="15" fill="1" visible="yes" active="no"/>
-<layer number="25" name="tNames" color="7" fill="1" visible="yes" active="no"/>
-<layer number="26" name="bNames" color="7" fill="1" visible="yes" active="no"/>
-<layer number="27" name="tValues" color="7" fill="1" visible="yes" active="no"/>
-<layer number="28" name="bValues" color="7" fill="1" visible="yes" active="no"/>
+<layer number="1" name="Top" color="4" fill="1" visible="no" active="no"/>
+<layer number="16" name="Bottom" color="1" fill="1" visible="no" active="no"/>
+<layer number="17" name="Pads" color="2" fill="1" visible="no" active="no"/>
+<layer number="18" name="Vias" color="2" fill="1" visible="no" active="no"/>
+<layer number="19" name="Unrouted" color="6" fill="1" visible="no" active="no"/>
+<layer number="20" name="Dimension" color="24" fill="1" visible="no" active="no"/>
+<layer number="21" name="tPlace" color="7" fill="1" visible="no" active="no"/>
+<layer number="22" name="bPlace" color="7" fill="1" visible="no" active="no"/>
+<layer number="23" name="tOrigins" color="15" fill="1" visible="no" active="no"/>
+<layer number="24" name="bOrigins" color="15" fill="1" visible="no" active="no"/>
+<layer number="25" name="tNames" color="7" fill="1" visible="no" active="no"/>
+<layer number="26" name="bNames" color="7" fill="1" visible="no" active="no"/>
+<layer number="27" name="tValues" color="7" fill="1" visible="no" active="no"/>
+<layer number="28" name="bValues" color="7" fill="1" visible="no" active="no"/>
 <layer number="29" name="tStop" color="7" fill="3" visible="no" active="no"/>
 <layer number="30" name="bStop" color="7" fill="6" visible="no" active="no"/>
@@
 <layer number="35" name="tGlue" color="7" fill="4" visible="no" active="no"/>
 <layer number="36" name="bGlue" color="7" fill="5" visible="no" active="no"/>
-<layer number="37" name="tTest" color="7" fill="1" visible="yes" active="no"/>
-<layer number="38" name="bTest" color="7" fill="1" visible="yes" active="no"/>
+<layer number="37" name="tTest" color="7" fill="1" visible="no" active="no"/>
+<layer number="38" name="bTest" color="7" fill="1" visible="no" active="no"/>
 <layer number="39" name="tKeepout" color="4" fill="11" visible="no" active="no"/>
 <layer number="40" name="bKeepout" color="1" fill="11" visible="no" active="no"/>
@@
 <layer number="44" name="Drills" color="7" fill="1" visible="no" active="no"/>
 <layer number="45" name="Holes" color="7" fill="1" visible="no" active="no"/>
-<layer number="46" name="Milling" color="3" fill="1" visible="yes" active="no"/>
-<layer number="47" name="Measures" color="7" fill="1" visible="yes" active="no"/>
-<layer number="48" name="Document" color="7" fill="1" visible="yes" active="no"/>
-<layer number="49" name="Reference" color="7" fill="1" visible="yes" active="no"/>
-<layer number="50" name="dxf" color="7" fill="1" visible="yes" active="no"/>
-<layer number="51" name="tDocu" color="7" fill="1" visible="yes" active="no"/>
-<layer number="52" name="bDocu" color="7" fill="1" visible="yes" active="no"/>
-<layer number="53" name="tGND_GNDA" color="7" fill="9" visible="yes" active="no"/>
-<layer number="54" name="bGND_GNDA" color="1" fill="9" visible="yes" active="no"/>
-<layer number="56" name="wert" color="7" fill="1" visible="yes" active="no"/>
-<layer number="57" name="tCAD" color="7" fill="1" visible="yes" active="no"/>
-<layer number="58" name="bCAD" color="11" fill="1" visible="yes" active="no"/>
-<layer number="59" name="tCarbon" color="7" fill="1" visible="yes" active="no"/>
-<layer number="60" name="bCarbon" color="7" fill="1" visible="yes" active="no"/>
+<layer number="46" name="Milling" color="3" fill="1" visible="no" active="no"/>
+<layer number="47" name="Measures" color="7" fill="1" visible="no" active="no"/>
+<layer number="48" name="Document" color="7" fill="1" visible="no" active="no"/>
+<layer number="49" name="Reference" color="7" fill="1" visible="no" active="no"/>
+<layer number="50" name="dxf" color="7" fill="1" visible="no" active="no"/>
+<layer number="51" name="tDocu" color="7" fill="1" visible="no" active="no"/>
+<layer number="52" name="bDocu" color="7" fill="1" visible="no" active="no"/>
+<layer number="53" name="tGND_GNDA" color="7" fill="9" visible="no" active="no"/>
+<layer number="54" name="bGND_GNDA" color="1" fill="9" visible="no" active="no"/>
+<layer number="56" name="wert" color="7" fill="1" visible="no" active="no"/>
+<layer number="57" name="tCAD" color="7" fill="1" visible="no" active="no"/>
+<layer number="58" name="bCAD" color="11" fill="1" visible="no" active="no"/>
+<layer number="59" name="tCarbon" color="7" fill="1" visible="no" active="no"/>
+<layer number="60" name="bCarbon" color="7" fill="1" visible="no" active="no"/>
 <layer number="88" name="SimResults" color="9" fill="1" visible="yes" active="yes"/>
 <layer number="89" name="SimProbes" color="9" fill="1" visible="yes" active="yes"/>
@@
 <part name="U$56" library="microbuilder" deviceset="3.3V" device=""/>
 <part name="U$57" library="microbuilder" deviceset="3.3V" device=""/>
-<part name="R24" library="microbuilder" deviceset="RESISTOR_4PACK" device="" value="100k"/>
+<part name="R24" library="microbuilder" deviceset="RESISTOR_4PACK" device="" value="10k"/>
 <part name="U$17" library="microbuilder" deviceset="3.3V" device=""/>
 <part name="D4" library="microbuilder" deviceset="DIODE-SCHOTTKY" device="SOD-123" value="MBR120"/>
@@
 <net name="SDA" class="0">
 <segment>
-<wire x1="40.64" y1="27.94" x2="53.34" y2="27.94" width="0.1524" layer="91"/>
-<label x="43.18" y="27.94" size="1.778" layer="95"/>
-<pinref part="X8" gate="G$1" pin="IO23"/>
-</segment>
-<segment>
 <pinref part="R13" gate="G$1" pin="2"/>
 <wire x1="71.12" y1="52.07" x2="69.342" y2="52.07" width="0.1524" layer="91"/>
@@
 <label x="-91.44" y="40.64" size="1.778" layer="95"/>
 <pinref part="U3" gate="G$1" pin="SDA"/>
+</segment>
+<segment>
+<wire x1="40.64" y1="33.02" x2="53.34" y2="33.02" width="0.1524" layer="91"/>
+<label x="43.18" y="33.02" size="1.778" layer="95"/>
+<pinref part="X8" gate="G$1" pin="IO21"/>
 </segment>
 </net>
@@
 <net name="NEOPIX" class="0">
 <segment>
-<wire x1="40.64" y1="33.02" x2="53.34" y2="33.02" width="0.1524" layer="91"/>
-<label x="43.18" y="33.02" size="1.778" layer="95"/>
-<pinref part="X8" gate="G$1" pin="IO21"/>
-</segment>
-<segment>
 <wire x1="142.748" y1="-25.146" x2="130.048" y2="-25.146" width="0.1524" layer="91"/>
 <pinref part="LED1" gate="G$1" pin="DI"/>
 <label x="127.508" y="-25.146" size="1.778" layer="95"/>
+</segment>
+<segment>
+<wire x1="40.64" y1="27.94" x2="53.34" y2="27.94" width="0.1524" layer="91"/>
+<label x="43.18" y="27.94" size="1.778" layer="95"/>
+<pinref part="X8" gate="G$1" pin="IO23"/>
 </segment>
 </net>
@@
 </segment>
 </net>
-<net name="!RST_3V" class="0">
-<segment>
-<pinref part="U3" gate="G$1" pin="!RST"/>
-<wire x1="-93.98" y1="33.02" x2="-86.36" y2="33.02" width="0.1524" layer="91"/>
-<wire x1="-86.36" y1="45.72" x2="-86.36" y2="33.02" width="0.1524" layer="91"/>
-<pinref part="R24" gate="G$2" pin="1"/>
-</segment>
-</net>
-<net name="!WAKE_3V" class="0">
+<net name="WAKE_CCS811" class="0">
 <segment>
 <pinref part="U3" gate="G$1" pin="!WAKE"/>
@@
 <wire x1="-81.28" y1="45.72" x2="-81.28" y2="35.56" width="0.1524" layer="91"/>
 <pinref part="R24" gate="G$3" pin="1"/>
+<label x="-77.216" y="35.306" size="1.778" layer="95" rot="R90"/>
+</segment>
+<segment>
+<pinref part="X8" gate="G$1" pin="IO13/A2_4"/>
+<wire x1="40.64" y1="50.8" x2="53.34" y2="50.8" width="0.1524" layer="91"/>
+<label x="43.18" y="50.8" size="1.778" layer="95"/>
 </segment>
 </net>
@@
 </segment>
 </net>
+<net name="RST_CCS811" class="0">
+<segment>
+<pinref part="U3" gate="G$1" pin="!RST"/>
+<wire x1="-93.98" y1="33.02" x2="-86.36" y2="33.02" width="0.1524" layer="91"/>
+<wire x1="-86.36" y1="45.72" x2="-86.36" y2="33.02" width="0.1524" layer="91"/>
+<pinref part="R24" gate="G$2" pin="1"/>
+<label x="-91.186" y="32.512" size="1.778" layer="95"/>
+</segment>
+<segment>
+<pinref part="X8" gate="G$1" pin="IO14/A2_6"/>
+<wire x1="40.64" y1="48.26" x2="53.34" y2="48.26" width="0.1524" layer="91"/>
+<label x="43.18" y="48.514" size="1.778" layer="95"/>
+</segment>
+</net>
+<net name="INT_CCS811" class="0">
+<segment>
+<pinref part="U3" gate="G$1" pin="!INT"/>
+<wire x1="-93.98" y1="30.48" x2="-90.678" y2="30.48" width="0.1524" layer="91"/>
+<label x="-94.234" y="30.48" size="1.778" layer="95"/>
+</segment>
+<segment>
+<pinref part="X8" gate="G$1" pin="IO15/A2_3"/>
+<wire x1="40.64" y1="45.72" x2="53.086" y2="45.72" width="0.1524" layer="91"/>
+<label x="43.18" y="45.72" size="1.778" layer="95"/>
+</segment>
+</net>

Commit message: v2
Parts:
- removed C8: DSK-3R3H224U-HL, DSK-3R3H224U-HL:DSK-3R3H224U-HL
- added 3V3: SM02B-GHS-TB_LF__SN_, SM02B-GHS-TB_LF__SN_:SM02B-GHS-TB_LF__SN_
- added C11: 1uF, microbuilder:CAP_CERAMIC0603_NO
- added C12: 10µF, microbuilder:CAP_CERAMIC0805-NOOUTLINE
- added R18: 100K, microbuilder:RESISTOR_0603_NOOUT
- added U1: AP2112-3.3, microbuilder:VREG_SOT23-5
- R3: value 5K -> 10K
Connections:
- new net 3.3V-2: 3V3.2, C11.1, C12.1, C30.1, IC4G$1.REGIN, IC4G$1.VDD, IC4G$1.VIO, LED1.VDD, R24G$1.2, R24G$2.2, R24G$3.2, R46G$3.1, U1.OUT, U3.VDD
- new net EN_U1: R18.1, U1.EN
- net 3.3V: now also R3.1; no longer C30.1, C8.1, IC4G$1.REGIN, IC4G$1.VDD, IC4G$1.VIO, LED1.VDD, OK1.COL, R24G$1.2, R24G$2.2, R24G$3.2, R46G$3.1, U3.VDD
- net GND: now also 3V3.1, 3V3.3, 3V3.4, C11.2, C12.2, OK1.EMIT, U1.GND; no longer C8.2, R3.1
- net ISO_DIN: now also OK1.COL; no longer OK1.EMIT
- net VBUS: now also R18.2, U1.IN
Other:
- moved on the sheet: R3
